File: kicraft/server/sample_projects/weather-sensor/BMP280_QWIIC_USB_C.kicad_sch (KiCad schematic)
At the start: 0 parts

Commit message: feat(showcase): refresh landing samples from self-eval 20260614
Promote the three best boards from self-eval batch 20260614T215540Z
(all grade B) into the landing-page showcase, replacing the regressed
PIR night light (D/45, hit erc_errors + unprogrammable_mcu gates):

- usb-pd-trigger (NEW, featured hero) — 81.0, fab-ready
- weather-sensor (re-promoted; stem A_BMP280_BAROMETRIC -> BMP280_QWIIC_USB_C)
- bench-breakout (re-promoted; 4->5 sheets, 16->19 parts)

Regenerated board.png/hero.png renders and interactive board.glb models
via scripts/promote_to_sample.py. Already live (deploy/restart-web.sh).

Co-Authored-By: Claude Opus 4.8 (1M context) <noreply@anthropic.com>
Other:
- title: Build a BMP280 barometric weather sensor breakout board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 -> A BMP280 barometric pressure sensor board with Qwiic/STEMMA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
Changed lines of the file:
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@@
 	(paper "A4")
 	(title_block
-		(title "Build a BMP280 barometric weather sensor breakout board…")
+		(title "A BMP280 barometric pressure sensor board with Qwiic/STEMMA…")
 		(rev "1.0")
 		(comment 1 "Generated by KiCraft pipeline")
@@
 		)
 		(instances
-			(project "A_BMP280_BAROMETRIC"
+			(project "BMP280_QWIIC_USB_C"
 				(path "/" (page "POWER"))
 			)
@@
 		)
 		(instances
-			(project "A_BMP280_BAROMETRIC"
+			(project "BMP280_QWIIC_USB_C"
 				(path "/" (page "SENSOR"))
 			)
